File: snake-pcb/snake-pcb.kicad_pcb (KiCad board)
At the start: 4 copper layers, 228.2 x 80.6 mm, 199 parts, among them J1 USB_C, J2 Conn_01x05_Socket, SW1 SW_Push, SW2 RotaryEncoder_Switch, U1 STM32F072CBT6, U3 XC6206, U4 USBLC6-2SC6

Commit message: pcb almost ever mo finished!
Other:
- board text added: "3.3V"
- board text added: "5V"
- board text added: "GND"
- board text added: "SCL"
- board text added: "SDA"
