File: snake-pcb/snake-pcb.kicad_sch (KiCad schematic)
At the start: 20 parts, among them J1 USB_C, SW1 SW_Push, U1 STM32F072CBT6, U3 XC6206, U4 USBLC6-2SC6

Commit message: pcb almost finished!
Parts:
- added CapLED1, CapLED10, CapLED11, CapLED12, CapLED13, CapLED14, CapLED15, CapLED16, CapLED17, CapLED18, CapLED19, CapLED2, CapLED20, CapLED21, CapLED22, CapLED23, CapLED24, CapLED25, CapLED26, CapLED27, CapLED28, CapLED29, CapLED3, CapLED30, CapLED31, CapLED32, CapLED33, CapLED34, CapLED35, CapLED36, CapLED37, CapLED38, CapLED39, CapLED4, CapLED40, CapLED41, CapLED42, CapLED43, CapLED5, CapLED6, CapLED7, CapLED8, CapLED9: 100nF, ScottoKeebs_Components:Capacitor_0402, symbol Device:C_Small
- added D1, D10, D11, D12, D13, D14, D15, D16, D17, D18, D19, D2, D20, D21, D22, D23, D24, D25, D26, D27, D28, D29, D3, D30, D31, D32, D33, D34, D35, D36, D37, D38, D39, D4, D40, D41, D42, D5, D6, D7, D8, D9, DLED1: 1N4148W, Diode_SMD:D_SOD-123, symbol Diode:1N4148W
- added J2: Conn_01x05_Socket, Connector_JST:JST_EH_B5B-EH-A_1x05_P2.50mm_Vertical, symbol Connector:Conn_01x05_Socket
- added LED1, LED10, LED11, LED12, LED13, LED14, LED15, LED16, LED17, LED18, LED19, LED2, LED20, LED21, LED22, LED23, LED24, LED25, LED26, LED27, LED28, LED29, LED3, LED30, LED31, LED32, LED33, LED34, LED35, LED36, LED37, LED38, LED39, LED4, LED40, LED41, LED42, LED43, LED5, LED6, LED7, LED8, LED9: SK6812MINI, ScottoKeebs_Components:LED_SK6812MINI, symbol LED:SK6812MINI
- added MX1, MX10, MX11, MX12, MX13, MX14, MX15, MX16, MX17, MX18, MX19, MX2, MX20, MX21, MX22, MX23, MX24, MX25, MX26, MX27, MX28, MX29, MX3, MX30, MX31, MX32, MX33, MX34, MX35, MX37, MX38, MX39, MX4, MX40, MX41, MX42, MX43, MX5, MX6, MX7, MX8, MX9: MX_SW_solder, PCM_marbastlib-mx:SW_MX_HS_CPG151101S11_1u, symbol PCM_marbastlib-mx:MX_SW_solder
- added MX36: MX_SW_solder, PCM_marbastlib-mx:SW_MX_HS_CPG151101S11_1.25u, symbol PCM_marbastlib-mx:MX_SW_solder
- added S35: MX_stab, PCM_marbastlib-mx:STAB_MX_P_ISO-ROT, symbol PCM_marbastlib-mx:MX_stab
- added S39: MX_stab, PCM_marbastlib-mx:STAB_MX_P_2.75u, symbol PCM_marbastlib-mx:MX_stab
- added S40: MX_stab, PCM_marbastlib-mx:STAB_MX_P_2.25u, symbol PCM_marbastlib-mx:MX_stab
- added S43: MX_stab, PCM_marbastlib-mx:STAB_MX_P_7u, symbol PCM_marbastlib-mx:MX_stab
- added SW2: RotaryEncoder_Switch, ScottoKeebs_Scotto:Encoder_EC11_MX, symbol Device:RotaryEncoder_Switch
Connections:
- net +3.3V: now also J2.5 (Pin_5)
- net +5V: now also CapLED10.2, CapLED11.2, CapLED12.2, CapLED13.2, CapLED14.2, CapLED15.2, CapLED16.2, CapLED17.2, CapLED18.2, CapLED19.2, CapLED2.2, CapLED20.2, CapLED21.2, CapLED22.2, CapLED23.2, CapLED24.2, CapLED25.2, CapLED26.2, CapLED27.2, CapLED28.2, CapLED29.2, CapLED3.2, CapLED30.2, CapLED31.2, CapLED32.2, CapLED33.2, CapLED34.2, CapLED35.2, CapLED36.2, CapLED37.2, CapLED38.2, CapLED39.2, CapLED4.2, CapLED40.2, CapLED41.2, CapLED42.2, CapLED43.2, CapLED5.2, CapLED6.2, CapLED7.2, CapLED8.2, CapLED9.2, DLED1.2 (A), J2.2 (Pin_2), LED10.4 (VDD), LED11.4 (VDD), LED12.4 (VDD), LED13.4 (VDD), LED14.4 (VDD), LED15.4 (VDD), LED16.4 (VDD), LED17.4 (VDD), LED18.4 (VDD), LED19.4 (VDD), LED2.4 (VDD), LED20.4 (VDD), LED21.4 (VDD), LED22.4 (VDD), LED23.4 (VDD), LED24.4 (VDD), LED25.4 (VDD), LED26.4 (VDD), LED27.4 (VDD), LED28.4 (VDD), LED29.4 (VDD), LED3.4 (VDD), LED30.4 (VDD), LED31.4 (VDD), LED32.4 (VDD), LED33.4 (VDD), LED34.4 (VDD), LED35.4 (VDD), LED36.4 (VDD), LED37.4 (VDD), LED38.4 (VDD), LED39.4 (VDD), LED4.4 (VDD), LED40.4 (VDD), LED41.4 (VDD), LED42.4 (VDD), LED43.4 (VDD), LED5.4 (VDD), LED6.4 (VDD), LED7.4 (VDD), LED8.4 (VDD), LED9.4 (VDD)
- net GND: now also CapLED1.1, CapLED10.1, CapLED11.1, CapLED12.1, CapLED13.1, CapLED14.1, CapLED15.1, CapLED16.1, CapLED17.1, CapLED18.1, CapLED19.1, CapLED2.1, CapLED20.1, CapLED21.1, CapLED22.1, CapLED23.1, CapLED24.1, CapLED25.1, CapLED26.1, CapLED27.1, CapLED28.1, CapLED29.1, CapLED3.1, CapLED30.1, CapLED31.1, CapLED32.1, CapLED33.1, CapLED34.1, CapLED35.1, CapLED36.1, CapLED37.1, CapLED38.1, CapLED39.1, CapLED4.1, CapLED40.1, CapLED41.1, CapLED42.1, CapLED43.1, CapLED5.1, CapLED6.1, CapLED7.1, CapLED8.1, CapLED9.1, J2.1 (Pin_1), LED1.2 (VSS), LED10.2 (VSS), LED11.2 (VSS), LED12.2 (VSS), LED13.2 (VSS), LED14.2 (VSS), LED15.2 (VSS), LED16.2 (VSS), LED17.2 (VSS), LED18.2 (VSS), LED19.2 (VSS), LED2.2 (VSS), LED20.2 (VSS), LED21.2 (VSS), LED22.2 (VSS), LED23.2 (VSS), LED24.2 (VSS), LED25.2 (VSS), LED26.2 (VSS), LED27.2 (VSS), LED28.2 (VSS), LED29.2 (VSS), LED3.2 (VSS), LED30.2 (VSS), LED31.2 (VSS), LED32.2 (VSS), LED33.2 (VSS), LED34.2 (VSS), LED35.2 (VSS), LED36.2 (VSS), LED37.2 (VSS), LED38.2 (VSS), LED39.2 (VSS), LED4.2 (VSS), LED40.2 (VSS), LED41.2 (VSS), LED42.2 (VSS), LED43.2 (VSS), LED5.2 (VSS), LED6.2 (VSS), LED7.2 (VSS), LED8.2 (VSS), LED9.2 (VSS), SW2.C
- net A14 renamed col9
- net col9: now also MX10.1, MX22.1, MX34.1, MX42.1, SW2.S2
- net A15 renamed col10
- net col10: now also MX11.1, MX23.1, MX35.1
- net A3 renamed rotA
- net rotA: now also SW2.A
- net A4 renamed rotB
- net rotB: now also SW2.B
- net A5 renamed row2
- net row2: now also D25.1 (K), D26.1 (K), D27.1 (K), D28.1 (K), D29.1 (K), D30.1 (K), D31.1 (K), D32.1 (K), D33.1 (K), D34.1 (K)
- net A6 renamed row3
- net row3: now also D35.1 (K), D36.1 (K), D37.1 (K), D38.1 (K), D39.1 (K), D40.1 (K), D41.1 (K), D42.1 (K)
- net A7 renamed data 3.3v
- net data 3.3v: now also LED1.3 (DIN)
- net B0 renamed col0
- net col0: now also MX1.1, MX13.1, MX25.1, MX36.1
- net B1 renamed col1
- net col1: now also MX14.1, MX2.1, MX26.1, MX37.1
- net B10 renamed col3
- net col3: now also MX16.1, MX28.1, MX4.1
- net B11 renamed col4
- net col4: now also MX17.1, MX29.1, MX39.1, MX43.1, MX5.1
- net B12 renamed col5
- net col5: now also MX18.1, MX30.1, MX6.1
- net B13 renamed row0
- net row0: now also D1.1 (K), D10.1 (K), D11.1 (K), D12.1 (K), D2.1 (K), D3.1 (K), D4.1 (K), D5.1 (K), D6.1 (K), D7.1 (K), D8.1 (K), D9.1 (K)
- net B2 renamed col2
- net col2: now also MX15.1, MX27.1, MX3.1, MX38.1
- net B3 renamed col11
- net col11: now also MX12.1, MX24.1
- net B4 renamed row1
- net row1: now also D13.1 (K), D14.1 (K), D15.1 (K), D16.1 (K), D17.1 (K), D18.1 (K), D19.1 (K), D20.1 (K), D21.1 (K), D22.1 (K), D23.1 (K), D24.1 (K)
- net B5 renamed col8
- net col8: now also MX21.1, MX33.1, MX41.1, MX9.1
- net B6 renamed scl
- net scl: now also J2.4 (Pin_4)
- net B7 renamed sda
- net sda: now also J2.3 (Pin_3)
- net B8 renamed col6
- net col6: now also MX19.1, MX31.1, MX7.1
- net B9 renamed col7
- net col7: now also MX20.1, MX32.1, MX40.1, MX8.1
- new net: D14.2 (A), MX14.2
- new net: LED4.1 (DOUT), LED5.3 (DIN)
- new net: LED3.1 (DOUT), LED4.3 (DIN)
- new net: LED16.1 (DOUT), LED17.3 (DIN)
- new net: LED15.1 (DOUT), LED16.3 (DIN)
- new net: D27.2 (A), MX27.2
- new net: D7.2 (A), MX7.2
- new net: D30.2 (A), MX30.2
- new net: D40.2 (A), MX40.2
- new net: LED31.1 (DOUT), LED32.3 (DIN)
- new net: LED30.1 (DOUT), LED31.3 (DIN)
- new net: D31.2 (A), MX31.2
- new net: D23.2 (A), MX23.2
- new net: D21.2 (A), MX21.2
- new net: D12.2 (A), MX12.2
- new net: LED41.1 (DOUT), LED42.3 (DIN)
- new net: LED40.1 (DOUT), LED41.3 (DIN)
- new net: D11.2 (A), MX11.2
- new net: LED42.1 (DOUT), LED43.3 (DIN)
- new net: D41.2 (A), MX41.2
- new net: D38.2 (A), MX38.2
- new net: D20.2 (A), MX20.2
- new net: D22.2 (A), MX22.2
- new net: LED29.1 (DOUT), LED30.3 (DIN)
- new net: LED36.1 (DOUT), LED37.3 (DIN)
- new net: LED35.1 (DOUT), LED36.3 (DIN)
- new net: D16.2 (A), MX16.2
- new net: D18.2 (A), MX18.2
- new net: LED14.1 (DOUT), LED15.3 (DIN)
- new net: D32.2 (A), MX32.2
- new net: D37.2 (A), MX37.2
- new net: LED17.1 (DOUT), LED18.3 (DIN)
- new net: D13.2 (A), MX13.2
- new net: LED10.1 (DOUT), LED11.3 (DIN)
- new net: LED10.3 (DIN), LED9.1 (DOUT)
- new net: LED7.1 (DOUT), LED8.3 (DIN)
- new net: LED6.1 (DOUT), LED7.3 (DIN)
- new net: D17.2 (A), MX17.2
- new net: D35.2 (A), MX35.2
- new net: D34.2 (A), MX34.2
- new net: D33.2 (A), MX33.2
- new net: LED23.1 (DOUT), LED24.3 (DIN)
- new net: LED22.1 (DOUT), LED23.3 (DIN)
- new net: D1.2 (A), MX1.2
- new net: LED20.1 (DOUT), LED21.3 (DIN)
- new net: LED19.1 (DOUT), LED20.3 (DIN)
- new net: LED33.1 (DOUT), LED34.3 (DIN)
- new net: LED32.1 (DOUT), LED33.3 (DIN)
- new net: LED39.1 (DOUT), LED40.3 (DIN)
- new net: LED38.1 (DOUT), LED39.3 (DIN)
- new net: D6.2 (A), MX6.2
- new net: LED21.1 (DOUT), LED22.3 (DIN)
- new net: D10.2 (A), MX10.2
- new net: D4.2 (A), MX4.2
- new net: LED37.1 (DOUT), LED38.3 (DIN)
- new net: D8.2 (A), MX8.2
- new net: D36.2 (A), MX36.2
- new net: LED28.1 (DOUT), LED29.3 (DIN)
- new net: LED34.1 (DOUT), LED35.3 (DIN)
- new net: D28.2 (A), MX28.2
- new net: D2.2 (A), MX2.2
- new net: D29.2 (A), MX29.2
- new net: LED18.1 (DOUT), LED19.3 (DIN)
- new net: LED2.1 (DOUT), LED3.3 (DIN)
- new net: D42.2 (A), MX42.2, SW2.S1
- new net: LED26.1 (DOUT), LED27.3 (DIN)
- new net: LED25.1 (DOUT), LED26.3 (DIN)
- new net: D24.2 (A), MX24.2
- new net: D5.2 (A), MX5.2
- new net: LED13.1 (DOUT), LED14.3 (DIN)
- new net: D15.2 (A), MX15.2
- new net: D26.2 (A), MX26.2
- new net: D9.2 (A), MX9.2
- new net: LED12.1 (DOUT), LED13.3 (DIN)
- new net: LED8.1 (DOUT), LED9.3 (DIN)
- new net: LED24.1 (DOUT), LED25.3 (DIN)
- new net: LED1.1 (DOUT), LED2.3 (DIN)
- new net: LED5.1 (DOUT), LED6.3 (DIN)
- new net: LED11.1 (DOUT), LED12.3 (DIN)
- new net: LED27.1 (DOUT), LED28.3 (DIN)
- new net: D19.2 (A), MX19.2
- new net: D3.2 (A), MX3.2
- new net: D25.2 (A), MX25.2
- new net DLED1_pwr: CapLED1.2, DLED1.1 (K), LED1.4 (VDD)
- new net d39: D39.2 (A), MX39.2, MX43.2
- no-connect marks 0 -> 1
